Commit message: Commit 18/04 - Implementati frames in tf2 - Aggiunto launch file per client e server

File: simulation_env/urdf/mogi_bot.urdf (robot description, URDF)
Before this commit: robot mogi_bot, 5 links, 4 joints
Links:
- link base_link: geometry collision box size=.4 .2 .1; collision sphere radius=0.0499
- link left_wheel: geometry collision cylinder length=.05 radius=.1; visual mesh filename=package://simulation_env/meshes/wheel.dae
- link right_wheel: geometry collision cylinder length=.05 radius=.1; visual mesh filename=package://simulation_env/meshes/wheel.dae
- link scan_link: geometry collision box size=.1 .1 .1; visual mesh filename=package://simulation_env/meshes/lidar.dae
